File: pcb/M,S/left.kicad_sch (KiCad schematic)
At the start: 57 parts, among them J1 USB_C_Receptacle_PowerOnly_6P, SW1 SW_Push, SW10 SW_Push, SW11 SW_Push, SW12 SW_Push, SW13 SW_Push, SW14 SW_Push, SW15 SW_Push, SW16 SW_Push, SW17 SW_Push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

Commit message: Modified M,S
Parts:
- removed BT1: Battery, axseem:JST_1.25mm_mid-mount, symbol Device:Battery
- removed J1: USB_C_Receptacle_PowerOnly_6P, axseem:USB-C_6Pin_Mid-mount, symbol Connector:USB_C_Receptacle_PowerOnly_6P
- removed JP1, JP2: Jumper_3P, axseem:SolderJumper-3_P, symbol Jumper:SolderJumper_3_Open
- removed RSW1: Reset_SW, axseem:TS-1289VE-4, symbol Switch:SW_Push
- added D47: D, Diode_SMD:D_SOD-323_HandSoldering, symbol Device:D
- added LBG1: BATT-, axseem:1pin_conn, symbol Lily58_Pro-rescue:i2c_pin-Lily58-cache
- added LBP1: BATT+, axseem:1pin_conn, symbol Lily58_Pro-rescue:i2c_pin-Lily58-cache
- added LDisplay1: nice!view, axseem:nice_view_1side, symbol niceview:nice!view
- added PWSW2: SW_SPDT_312, axseem:switch-MSK-12C02-smd, symbol Switch:SW_SPDT_312
- added RSW3: SW_RST, axseem:TACT_SWITCH_TVBP06, symbol Lily58_Pro-rescue:SW_RST-Lily58-cache
- added SW47: SW_Push, axseem:SW_MX_Choc-v1v2_Hotswap, symbol Switch:SW_Push
- U1: footprint axseem:ProMicro_SMD -> axseem:ProMicro_rev
Connections:
- net LCol 0: now also U1.7 (4/D4), SW47.1; no longer U1.5 (2/D1/SDA)
- net LCol 1: now also U1.8 (5/C6); no longer U1.6 (3/D0/SCL)
- net LCol 2: now also U1.9 (6/D7); no longer U1.7 (4/D4)
- net LCol 3: now also U1.10 (7/E6); no longer U1.8 (5/C6)
- net LCol 4: now also U1.11 (8/B4); no longer U1.9 (6/D7)
- net LCol 5: now also U1.12 (9/B5); no longer U1.10 (7/E6)
- net LGND: now also LBG1.1 (Pin_1), LDisplay1.4 (GND), RSW3.1
- net LRaw: now also PWSW2.2 (C)
- net LReset: now also RSW3.2
- net LRow 0: now also U1.16 (B1/15); no longer U1.12 (9/B5)
- net LRow 3: now also D47.1 (K)
- net LVCC: now also LDisplay1.3 (VCC)
- net LDATA: now reaches U1.1 (TX0/D3)
- net LDATA: now also LDisplay1.5 (CS)
- net LData: no longer names the net of U1.2 (RX1/D2)
- new net: LBP1.1 (Pin_1), PWSW2.3 (A)
- new net: D47.2 (A), SW47.2
- new net LSCL: LDisplay1.2 (SCK), U1.6 (3/D0/SCL)
- new net LSDA: LDisplay1.1 (MOSI), U1.5 (2/D1/SDA)
- no-connect marks 7 -> 6
Other:
- note removed: "Power"
- note removed: "Reset switch"
- note removed: "USB port"
