File: pcb/M,S/right.kicad_sch (KiCad schematic)
At the start: 57 parts, among them J2 USB_C_Receptacle_PowerOnly_6P, SW24 SW_Push, SW25 SW_Push, SW26 SW_Push, SW27 SW_Push, SW28 SW_Push, SW29 SW_Push, SW30 SW_Push, SW31 SW_Push, SW32 SW_Push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

Commit message: Modified M,S
Parts:
- removed BT2: Battery, axseem:JST_1.25mm_mid-mount, symbol Device:Battery
- removed J2: USB_C_Receptacle_PowerOnly_6P, axseem:USB-C_6Pin_Mid-mount, symbol Connector:USB_C_Receptacle_PowerOnly_6P
- removed JP3, JP4: Jumper_3P, axseem:SolderJumper-3_P, symbol Jumper:SolderJumper_3_Open
- removed RSW2: Reset_SW, axseem:TS-1289VE-4, symbol Switch:SW_Push
- added D48: D, Diode_SMD:D_SOD-323_HandSoldering, symbol Device:D
- added LDisplay2: nice!view, axseem:nice_view_1side, symbol niceview:nice!view
- added PWSW3: SW_SPDT_312, axseem:switch-MSK-12C02-smd, symbol Switch:SW_SPDT_312
- added RBG1: BATT-, axseem:1pin_conn, symbol Lily58_Pro-rescue:i2c_pin-Lily58-cache
- added RBP1: BATT+, axseem:1pin_conn, symbol Lily58_Pro-rescue:i2c_pin-Lily58-cache
- added RSW4: SW_RST, axseem:TACT_SWITCH_TVBP06, symbol Lily58_Pro-rescue:SW_RST-Lily58-cache
- added SW48: SW_Push, axseem:SW_MX_Choc-v1v2_Hotswap, symbol Switch:SW_Push
- U2: footprint axseem:ProMicro_SMD -> axseem:ProMicro_rev
Connections:
- net RCol 0: now also SW48.1
- net RGND: now also LDisplay2.4 (GND), RBG1.1 (Pin_1), RSW4.1
- net RRaw: now also PWSW3.2 (C)
- net RReset: now also RSW4.2
- net RRow 3: now also D48.1 (K)
- net RVCC: now also LDisplay2.3 (VCC)
- net RSDA: now reaches U2.5 (2/D1/SDA)
- net RSDA: now also LDisplay2.1 (MOSI)
- net RSCL: now reaches U2.6 (3/D0/SCL)
- net RSCL: now also LDisplay2.2 (SCK)
- net RData renamed RDATA
- net RDATA: now also LDisplay2.5 (CS)
- new net: D48.2 (A), SW48.2
- new net: PWSW3.1 (B), RBP1.1 (Pin_1)
- no-connect marks 7 -> 6
Other:
- note removed: "Power"
- note removed: "Reset switch"
- note removed: "USB port"
